Commit message: Sync to released robotis_manipulator

File: open_manipulator_description/urdf/open_manipulator.urdf.xacro (robot description, xacro)
@@ -43,5 +43,5 @@
       </geometry>
     </collision>
-    <inertial>
+<!--    <inertial>
       <origin xyz="0 0 0" />
       <mass value="0.082" />
@@ -49,6 +49,6 @@
                iyy="0.1" iyz="0.0"
                izz="0.1" />
-    </inertial>
-    <!-- <inertial>
+    </inertial>-->
+     <inertial>
       <origin xyz="3.0876154e-04 0.0000000e+00 -1.2176461e-04" />
       <mass value="7.9119962e-02" />
@@ -56,5 +56,5 @@
                iyy="2.1898364e-05" iyz="0.0"
                izz="1.9267361e-05" />
-    </inertial> -->
+    </inertial>
   </link>
   <!-- Joint 1 -->
@@ -71,5 +71,5 @@
   <link name="link2">
     <visual>
-      <origin xyz="0 0 0.018" rpy="0 0 0"/>
+      <origin xyz="0 0 0.019" rpy="0 0 0"/>
       <geometry>
         <mesh filename="package://open_manipulator_description/meshes/chain_link2.stl" scale="0.001 0.001 0.001"/>
@@ -78,10 +78,10 @@
     </visual>
     <collision>
-      <origin xyz="0 0 0.018" rpy="0 0 0"/>
+      <origin xyz="0 0 0.019" rpy="0 0 0"/>
       <geometry>
         <mesh filename="package://open_manipulator_description/meshes/chain_link2.stl" scale="0.001 0.001 0.001"/>
       </geometry>
     </collision>
-    <inertial>
+<!--    <inertial>
       <origin xyz="0 0 0" />
       <mass value="0.098" />
@@ -89,6 +89,6 @@
                iyy="0.1" iyz="0.0"
                izz="0.1" />
-    </inertial>
-    <!-- <inertial>
+    </inertial>-->
+     <inertial>
       <origin xyz="-3.0184870e-04 5.4043684e-04 ${0.018 + 2.9433464e-02}" />
       <mass value="9.8406837e-02" />
@@ -96,5 +96,5 @@
                iyy="3.2689329e-05" iyz="2.8511935e-08"
                izz="1.8850320e-05" />
-    </inertial> -->
+    </inertial>
   </link>
   <!--  Joint 2 -->
@@ -102,5 +102,5 @@
     <parent link="link2"/>
     <child link="link3"/>
-    <origin xyz="0.0 0.0 0.058" rpy="0 0 0"/>
+    <origin xyz="0.0 0.0 0.0595" rpy="0 0 0"/>
     <axis xyz="0 1 0"/>
     <limit velocity="4.8" effort="1" lower="${-pi*0.57}" upper="${pi*0.5}" />
@@ -123,5 +123,5 @@
       </geometry>
     </collision>
-    <inertial>
+<!--    <inertial>
       <origin xyz="0 0 0" />
       <mass value="0.136" />
@@ -129,6 +129,6 @@
                iyy="0.1" iyz="0.0"
                izz="0.1" />
-    </inertial>
-    <!-- <inertial>
+    </inertial>-->
+     <inertial>
       <origin xyz="1.0308393e-02 3.7743363e-04 1.0170197e-01" />
       <mass value="1.3850917e-01" />
@@ -136,5 +136,5 @@
                iyy="3.4290447e-04" iyz="-1.5717516e-06"
                izz="6.0346498e-05" />
-    </inertial> -->
+    </inertial>
   </link>
   <!--  Joint 3 -->
@@ -163,5 +163,5 @@
       </geometry>
     </collision>
-    <inertial>
+<!--    <inertial>
       <origin xyz="0 0 0" />
       <mass value="0.131" />
@@ -169,6 +169,6 @@
                iyy="0.1" iyz="0.0"
                izz="0.1" />
-    </inertial>
-    <!-- <inertial>
+    </inertial>-->
+     <inertial>
       <origin xyz="9.0909590e-02 3.8929816e-04 2.2413279e-04" />
       <mass value="1.3274562e-01" />
@@ -176,5 +176,5 @@
                iyy="2.4230292e-04" iyz="1.1559550e-08"
                izz="2.5155057e-04" />
-    </inertial> -->
+    </inertial>
   </link>
   <!--  Joint 4 -->
@@ -203,5 +203,5 @@
       </geometry>
     </collision>
-    <inertial>
+<!--    <inertial>
       <origin xyz="0 0 0" />
       <mass value="0.141" />
@@ -209,6 +209,6 @@
                iyy="0.1" iyz="0.0"
                izz="0.1" />
-    </inertial>
-    <!-- <inertial>
+    </inertial>-->
+     <inertial>
       <origin xyz="4.4206755e-02 3.6839985e-07 8.9142216e-03" />
       <mass value="1.4327573e-01" />
@@ -216,5 +216,5 @@
                iyy="7.5980465e-05" iyz="0.0"
                izz="9.3127351e-05" />
-    </inertial> -->
+    </inertial>
   </link>
   <!--  Gripper link -->
@@ -236,9 +236,9 @@
       <origin xyz="0 0 0" />
       <mass value="0.017" />
-      <inertia ixx="0.1" ixy="0.0" ixz="0.0"
-               iyy="0.1" iyz="0.0"
-               izz="0.1" />
-    </inertial>
-    <!-- <inertial>
+      <inertia ixx="1.0e-03" ixy="0.0" ixz="0.0"
+               iyy="1.0e-03" iyz="0.0"
+               izz="1.0e-03" />
+    </inertial>
+<!--     <inertial>
       <origin xyz="${0.028 + 8.3720668e-03} ${0.0246 + 9.9696160e-03} -4.2836895e-07" />
       <mass value="3.2218127e-02" />
@@ -246,5 +246,5 @@
                iyy="2.2552871e-05" iyz="-3.1463634e-10"
                izz="1.7605306e-05" />
-    </inertial> -->
+    </inertial>-->
   </link>
   <!--  Gripper joint -->
@@ -252,5 +252,5 @@
     <parent link="link5"/>
     <child link="gripper_link"/>
-    <origin xyz="0.0817 0.019 0.0" rpy="0 0 0"/>
+    <origin xyz="0.0817 0.021 0.0" rpy="0 0 0"/>
     <axis xyz="0 1 0"/>
     <limit velocity="4.8" effort="1" lower="-0.010" upper="0.019" />
@@ -276,9 +276,9 @@
       <origin xyz="0 0 0" />
       <mass value="0.017" />
-      <inertia ixx="0.1" ixy="0.0" ixz="0.0"
-               iyy="0.1" iyz="0.0"
-               izz="0.1" />
-    </inertial>
-    <!-- <inertial>
+      <inertia ixx="1.0e-03" ixy="0.0" ixz="0.0"
+               iyy="1.0e-03" iyz="0.0"
+               izz="1.0e-03" />
+    </inertial>
+<!--     <inertial>
       <origin xyz="${0.028 + 8.3720668e-03} ${-0.0246 - 9.9696160e-03} -4.2836895e-07" />
       <mass value="3.2218127e-02" />
@@ -286,5 +286,5 @@
                iyy="2.2552871e-05" iyz="-3.1463634e-10"
                izz="1.7605306e-05" />
-    </inertial> -->
+    </inertial>-->
   </link>
   <!--  Gripper joint sub -->
@@ -292,5 +292,5 @@
     <parent link="link5"/>
     <child link="gripper_link_sub"/>
-    <origin xyz="0.0817 -0.019 0" rpy="0 0 0"/>
+    <origin xyz="0.0817 -0.021 0" rpy="0 0 0"/>
     <axis xyz="0 -1 0"/>
     <limit velocity="4.8" effort="1" lower="-0.010" upper="0.019" />
@@ -301,5 +301,5 @@
   <!-- end effector joint -->
   <joint name="end_effector_joint" type="fixed">
-    <origin xyz="0.130 0.0 0.0" rpy="0 0 0"/>
+    <origin xyz="0.126 0.0 0.0" rpy="0 0 0"/>
     <parent link="link5"/>
     <child link="end_effector_link"/>
@@ -317,5 +317,5 @@
       <origin xyz="0.0 0.0 0.0" rpy="0 0 0"/>
       <mass value="0.001"/>
-      <inertia ixx="1.0" ixy="0.0" ixz="0.0" iyy="1.0" iyz="0.0" izz="1.0" />
+      <inertia ixx="1.0e-06" ixy="0.0" ixz="0.0" iyy="1.0e-06" iyz="0.0" izz="1.0e-06" />
     </inertial>
   </link>
