Commit message: change to xacro

File: open_manipulator_x_description/urdf/open_manipulator_x_robot.urdf.xacro (robot description, xacro)
@@ -8,35 +8,11 @@
   <!-- Import Transmission -->
   <xacro:include filename="$(find open_manipulator_x_description)/urdf/open_manipulator_x.transmission.xacro" />
-  <!-- Import URDF -->
-  <xacro:include filename="$(find open_manipulator_x_description)/urdf/open_manipulator_x.urdf.xacro" />
-  <!-- World -->
-  <link name="world"/>
-  <!-- World fixed joint-->
-  <joint name="world_fixed" type="fixed">
-    <origin xyz="0 0 0" rpy="0 0 0"/>
-    <parent link="world"/>
-    <child link="link1"/>
-  </joint>
-  <!-- !!!!!!!!!!!!!!!!!!!!!!!!!!!!!!!! -->
-  <!-- TODO:Xacro files do not work yet -->
-  <!-- !!!!!!!!!!!!!!!!!!!!!!!!!!!!!!!! -->
-  <material name="black">
-    <color rgba="0.0 0.0 0.0 1.0"/>
-  </material>
-  <material name="white">
-    <color rgba="1.0 1.0 1.0 1.0"/>
-  </material>
-  <material name="red">
-    <color rgba="0.8 0.0 0.0 1.0"/>
-  </material>
-  <material name="blue">
-    <color rgba="0.0 0.0 0.8 1.0"/>
-  </material>
-  <material name="green">
-    <color rgba="0.0 0.8 0.0 1.0"/>
-  </material>
-  <material name="grey">
-    <color rgba="0.5 0.5 0.5 1.0"/>
-  </material>
+  <xacro:macro name="open_manipulator_x" params="parent *origin">
+    <joint name="origin_to_link1" type="fixed">
+      <xacro:insert_block name="origin" />
+      <parent link="${parent}" />
+      <child link="link1" />
+      <axis xyz="0 0 1" />
+    </joint>
   <!-- Link 1 -->
   <link name="link1">
@@ -280,3 +256,4 @@
   </joint>
   <link name="camera_link"/>
+  </xacro:macro>
 </robot>

Commit message: adjust joint limits

File: open_manipulator_x_description/urdf/open_manipulator_x_robot.urdf.xacro (robot description, xacro)
@@ -44,5 +44,5 @@
     <origin xyz="0.012 0.0 0.017" rpy="0 0 0"/>
     <axis xyz="0 0 1"/>
-    <limit velocity="4.8" effort="1" lower="-2.82743338823" upper="2.82743338823" />
+    <limit velocity="4.8" effort="1" lower="-1.5708" upper="1.5708" />
   </joint>
   <!--  Link 2 -->
@@ -75,5 +75,5 @@
     <origin xyz="0.0 0.0 0.0595" rpy="0 0 0"/>
     <axis xyz="0 1 0"/>
-    <limit velocity="4.8" effort="1" lower="-1.79070781255" upper="1.57079632679" />
+    <limit velocity="4.8" effort="1" lower="0.0" upper="2.0" />
   </joint>
   <!--  Link 3 -->
@@ -106,5 +106,5 @@
     <origin xyz="0.024 0 0.128" rpy="0 0 0"/>
     <axis xyz="0 1 0"/>
-    <limit velocity="4.8" effort="1" lower="-0.94247779607" upper="1.38230076758" />
+    <limit velocity="4.8" effort="1" lower="-2.0" upper="1.38230076758" />
   </joint>
   <!--  Link 4 -->
@@ -137,5 +137,5 @@
     <origin xyz="0.124 0.0 0.0" rpy="0 0 0"/>
     <axis xyz="0 1 0"/>
-    <limit velocity="4.8" effort="1" lower="-1.79070781255" upper="2.04203522483" />
+    <limit velocity="4.8" effort="1" lower="-0.7" upper="2.04203522483" />
   </joint>
   <!--  Link 5 -->
